File: converter.kicad_pcb (KiCad board)
At the start: 2 copper layers, 91.4 x 34.3 mm, 53 parts, among them J1 USB-FOO, P1 OW1_5V, P10 OW3, P11 OW3_GND, P12 Front+, P13 Back+, P14 Front-, P15 Back-, P2 OW1, P3 OW1_GND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

Commit message: Improved ground routing, fixed one error
The error was a missing VCC connection at the back converter's input
Parts:
- U2: value LT1117-5.0 -> LM1117E
- moved R5 2.68 mm to (98.8, 110.0)
Connections:
- Q2 pad 3: N-000006 (its old number) -> +12V
- Q3 pad 3: N-000006 (its old number) -> +12V
- R3 pad 2: N-000006 (its old number) -> +12V
Routing:
- net +12V: track 81.2 -> 127.7 mm, vias 2 -> 4
- net GND: track 290.0 -> 309.2 mm, vias 4 -> 6
- net N-000006 (its old number): track 7.20 -> 0.00 mm
- net /back_pos: track 26.8 -> 28.2 mm, vias 1 -> 0
- net /front_neg: track 43.8 -> 42.7 mm
- net N-0000014: track 56.8 -> 57.3 mm
- net /back_neg: track 27.0 -> 26.6 mm, vias 2 -> 1
Other:
- net class Default: trace_width 0.254 -> 0.4064
- net class POWER added: clearance 0.254, trace_width 0.8128, via_dia 0.889, via_drill 0.635

Commit message: Added some info on the back silkscreen
Parts:
- added G***: OSHW-logo_silkscreen-back_8mm, OSHW-logo_silkscreen-back_8mm, B.Cu at (101.0, 95.9)
Other:
- board text added: "(c) 2014 by jaseg"
- board text added: "Bikelights"
- board text added: "CC-BY-SA"
- board text added: "Released under Creative Commons"
- board text added: "jaseg.net/bikelights.html"
Changed lines of the file:
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@@
     (area 26.619999 87.5538 118.4402 122.991033)
     (thickness 1.6)
-    (drawings 4)
+    (drawings 9)
     (tracks 358)
     (zones 0)
-    (modules 53)
+    (modules 54)
     (nets 29)
   )
@@
     (visible_elements FFFFFFBF)
     (pcbplotparams
-      (layerselection 32769)
+      (layerselection 284196865)
       (usegerberextensions true)
       (excludeedgelayer true)
@@
       (drillshape 0)
       (scaleselection 1)
-      (outputdirectory ../../../../tmp/))
+      (outputdirectory gerber/))
   )
   (net 0 "")
@@
     )
   )
+  (module OSHW-logo_silkscreen-back_8mm (layer B.Cu)
+    (at 100.965 95.885)
+    (fp_text reference G*** (at 0 -4.2418) (layer B.SilkS) hide
+      (effects (font (size 0.36322 0.36322) (thickness 0.07112)) (justify mirror))
+    )
+    (fp_text value OSHW-logo_silkscreen-back_8mm (at 0 4.2418) (layer B.SilkS) hide
+      (effects (font (size 0.36322 0.36322) (thickness 0.07112)) (justify mirror))
+    )
+    (fp_poly (pts (xy 2.42316 3.59156) (xy 2.38252 3.57124) (xy 2.28854 3.51282) (xy 2.15392 3.42392)
+      (xy 1.99644 3.31978) (xy 1.83896 3.21056) (xy 1.70942 3.1242) (xy 1.61798 3.06578)
+      (xy 1.57988 3.04546) (xy 1.55956 3.05054) (xy 1.48336 3.08864) (xy 1.37414 3.14452)
+      (xy 1.31064 3.17754) (xy 1.21158 3.22072) (xy 1.16078 3.23088) (xy 1.15316 3.21564)
+      (xy 1.11506 3.13944) (xy 1.05918 3.00736) (xy 0.98298 2.83464) (xy 0.89662 2.63144)
+      (xy 0.80264 2.413) (xy 0.7112 2.18948) (xy 0.6223 1.97612) (xy 0.54356 1.78562)
+      (xy 0.48006 1.63068) (xy 0.43942 1.52146) (xy 0.42418 1.47574) (xy 0.42926 1.46558)
+      (xy 0.48006 1.41732) (xy 0.56642 1.35128) (xy 0.75692 1.19634) (xy 0.94234 0.96266)
+      (xy 1.05664 0.6985) (xy 1.09474 0.40386) (xy 1.06172 0.13208) (xy 0.95504 -0.12954)
+      (xy 0.77216 -0.36576) (xy 0.55118 -0.54102) (xy 0.2921 -0.65278) (xy 0 -0.68834)
+      (xy -0.2794 -0.65786) (xy -0.5461 -0.55118) (xy -0.78232 -0.37084) (xy -0.88138 -0.25654)
+      (xy -1.01854 -0.01778) (xy -1.09728 0.23876) (xy -1.1049 0.30226) (xy -1.09474 0.5842)
+      (xy -1.01092 0.85344) (xy -0.8636 1.09474) (xy -0.65786 1.29032) (xy -0.62992 1.31064)
+      (xy -0.53594 1.38176) (xy -0.47244 1.43002) (xy -0.42164 1.47066) (xy -0.77978 2.33172)
+      (xy -0.83566 2.46888) (xy -0.93472 2.7051) (xy -1.02108 2.9083) (xy -1.08966 3.06832)
+      (xy -1.13792 3.17754) (xy -1.15824 3.22072) (xy -1.16078 3.22326) (xy -1.19126 3.22834)
+      (xy -1.2573 3.20294) (xy -1.37668 3.14452) (xy -1.45796 3.10388) (xy -1.5494 3.0607)
+      (xy -1.59004 3.04546) (xy -1.6256 3.06324) (xy -1.71196 3.12166) (xy -1.8415 3.20548)
+      (xy -1.9939 3.30962) (xy -2.14122 3.41122) (xy -2.27584 3.50012) (xy -2.3749 3.56108)
+      (xy -2.42316 3.58902) (xy -2.43078 3.58902) (xy -2.47142 3.56362) (xy -2.55016 3.50012)
+      (xy -2.667 3.38836) (xy -2.8321 3.2258) (xy -2.8575 3.2004) (xy -2.99466 3.0607)
+      (xy -3.10642 2.94386) (xy -3.18008 2.86258) (xy -3.20548 2.82448) (xy -3.20548 2.82448)
+      (xy -3.18262 2.77622) (xy -3.11912 2.6797) (xy -3.03022 2.54254) (xy -2.921 2.38252)
+      (xy -2.63652 1.9685) (xy -2.794 1.57734) (xy -2.84226 1.45796) (xy -2.90322 1.31318)
+      (xy -2.9464 1.20904) (xy -2.9718 1.16332) (xy -3.01244 1.14808) (xy -3.12166 1.12268)
+      (xy -3.2766 1.08966) (xy -3.45948 1.05664) (xy -3.63728 1.02362) (xy -3.7973 0.99314)
+      (xy -3.9116 0.97028) (xy -3.9624 0.96012) (xy -3.9751 0.9525) (xy -3.98526 0.9271)
+      (xy -3.99288 0.87376) (xy -3.99542 0.77724) (xy -3.99796 0.62484) (xy -3.99796 0.40386)
+      (xy -3.99796 0.381) (xy -3.99542 0.17018) (xy -3.99288 0.00254) (xy -3.9878 -0.10668)
+      (xy -3.98018 -0.14986) (xy -3.98018 -0.14986) (xy -3.92938 -0.16256) (xy -3.81762 -0.18542)
+      (xy -3.6576 -0.21844) (xy -3.4671 -0.254) (xy -3.45694 -0.25654) (xy -3.26644 -0.2921)
+      (xy -3.10896 -0.32512) (xy -2.9972 -0.35052) (xy -2.95148 -0.36576) (xy -2.94132 -0.37846)
+      (xy -2.90322 -0.45212) (xy -2.84734 -0.56896) (xy -2.78638 -0.71374) (xy -2.72288 -0.86106)
+      (xy -2.66954 -0.99568) (xy -2.63398 -1.09474) (xy -2.62382 -1.14046) (xy -2.62382 -1.14046)
+      (xy -2.65176 -1.18618) (xy -2.7178 -1.28524) (xy -2.80924 -1.41986) (xy -2.921 -1.58242)
+      (xy -2.92862 -1.59512) (xy -3.03784 -1.75514) (xy -3.12674 -1.88976) (xy -3.18516 -1.98628)
+      (xy -3.20548 -2.02946) (xy -3.20548 -2.032) (xy -3.16992 -2.08026) (xy -3.08864 -2.16916)
+      (xy -2.9718 -2.29108) (xy -2.8321 -2.43332) (xy -2.78638 -2.4765) (xy -2.63144 -2.6289)
+      (xy -2.52476 -2.72796) (xy -2.45618 -2.7813) (xy -2.42316 -2.794) (xy -2.42316 -2.79146)
+      (xy -2.3749 -2.76352) (xy -2.2733 -2.69748) (xy -2.13614 -2.6035) (xy -1.97358 -2.49428)
+      (xy -1.96342 -2.48666) (xy -1.8034 -2.37744) (xy -1.67132 -2.28854) (xy -1.5748 -2.22504)
+      (xy -1.53416 -2.19964) (xy -1.52654 -2.19964) (xy -1.46304 -2.21996) (xy -1.34874 -2.25806)
+      (xy -1.20904 -2.31394) (xy -1.06172 -2.37236) (xy -0.9271 -2.42824) (xy -0.8255 -2.4765)
+      (xy -0.77724 -2.5019) (xy -0.77724 -2.50444) (xy -0.75946 -2.56286) (xy -0.73152 -2.68224)
+      (xy -0.6985 -2.84734) (xy -0.6604 -3.04292) (xy -0.65532 -3.0734) (xy -0.61976 -3.2639)
+      (xy -0.58928 -3.42138) (xy -0.56642 -3.5306) (xy -0.55372 -3.57632) (xy -0.52832 -3.5814)
+      (xy -0.43434 -3.58902) (xy -0.2921 -3.59156) (xy -0.11938 -3.5941) (xy 0.06096 -3.59156)
+      (xy 0.23622 -3.58902) (xy 0.38862 -3.58394) (xy 0.4953 -3.57632) (xy 0.54102 -3.56616)
+      (xy 0.54356 -3.56362) (xy 0.5588 -3.5052) (xy 0.5842 -3.38582) (xy 0.61976 -3.22072)
+      (xy 0.65786 -3.0226) (xy 0.66294 -2.98958) (xy 0.6985 -2.79908) (xy 0.73152 -2.64414)
+      (xy 0.75438 -2.53492) (xy 0.76708 -2.49428) (xy 0.78232 -2.48412) (xy 0.86106 -2.4511)
+      (xy 0.98806 -2.39776) (xy 1.14808 -2.33426) (xy 1.51384 -2.1844) (xy 1.96088 -2.49428)
+      (xy 2.00406 -2.52222) (xy 2.16408 -2.63144) (xy 2.2987 -2.72034) (xy 2.39014 -2.77876)
+      (xy 2.42824 -2.80162) (xy 2.43078 -2.79908) (xy 2.4765 -2.76098) (xy 2.5654 -2.67716)
+      (xy 2.68732 -2.55778) (xy 2.82702 -2.41808) (xy 2.93116 -2.31394) (xy 3.05562 -2.18694)
+      (xy 3.13436 -2.10312) (xy 3.17754 -2.04724) (xy 3.19278 -2.01422) (xy 3.1877 -1.9939)
+      (xy 3.15976 -1.94818) (xy 3.09372 -1.84912) (xy 3.00228 -1.71196) (xy 2.89306 -1.55448)
+      (xy 2.80162 -1.41986) (xy 2.7051 -1.27) (xy 2.6416 -1.16332) (xy 2.61874 -1.10998)
+      (xy 2.62382 -1.08712) (xy 2.65684 -1.00076) (xy 2.71018 -0.86614) (xy 2.77622 -0.70866)
+      (xy 2.9337 -0.35306) (xy 3.16738 -0.30988) (xy 3.30708 -0.28194) (xy 3.5052 -0.24384)
+      (xy 3.69316 -0.20828) (xy 3.9878 -0.14986) (xy 3.99796 0.93218) (xy 3.95224 0.9525)
+      (xy 3.90906 0.9652) (xy 3.79984 0.98806) (xy 3.6449 1.01854) (xy 3.45948 1.0541)
+      (xy 3.30454 1.08458) (xy 3.14452 1.11252) (xy 3.03276 1.13538) (xy 2.98196 1.14554)
+      (xy 2.96926 1.16332) (xy 2.92862 1.23952) (xy 2.87274 1.36144) (xy 2.81178 1.50876)
+      (xy 2.74828 1.65862) (xy 2.6924 1.79832) (xy 2.65176 1.905) (xy 2.63906 1.96088)
+      (xy 2.65938 2.00406) (xy 2.72034 2.0955) (xy 2.8067 2.22758) (xy 2.91338 2.38506)
+      (xy 3.0226 2.54254) (xy 3.1115 2.67716) (xy 3.175 2.77368) (xy 3.2004 2.81686)
+      (xy 3.1877 2.84734) (xy 3.12674 2.92354) (xy 3.00736 3.04546) (xy 2.8321 3.22072)
+      (xy 2.80162 3.24866) (xy 2.66192 3.38328) (xy 2.54254 3.4925) (xy 2.46126 3.56616)
+      (xy 2.42316 3.59156)) (layer B.SilkS) (width 0.00254))
+  )
+  (gr_text jaseg.net/bikelights.html (at 80.645 113.03) (layer B.SilkS)
+    (effects (font (size 2.54 2.54) (thickness 0.508)) (justify mirror))
+  )
+  (gr_text CC-BY-SA (at 95.25 107.315) (layer B.SilkS)
+    (effects (font (size 2.54 2.54) (thickness 0.508)) (justify mirror))
+  )
+  (gr_text "Released under Creative Commons" (at 71.755 102.87) (layer B.SilkS)
+    (effects (font (size 2.54 2.54) (thickness 0.508)) (justify mirror))
+  )
+  (gr_text "(c) 2014 by jaseg" (at 78.105 98.425) (layer B.SilkS)
+    (effects (font (size 2.54 2.54) (thickness 0.508)) (justify mirror))
+  )
+  (gr_text Bikelights (at 85.725 93.98) (layer B.SilkS)
+    (effects (font (size 2.54 2.54) (thickness 0.508)) (justify mirror))
+  )
   (gr_line (start 26.67 121.92) (end 26.67 87.63) (angle 90) (layer Edge.Cuts) (width 0.1))
